File: player-board.kicad_pcb (KiCad board)
At the start: 2 copper layers, 45 x 30 mm, 24 parts, among them J1 Conn_02x03_Odd_Even, J2 Conn_01x05, U1 AMS1117, U2 ESP32-PICO-D4

Commit message: Different footprint on ESP32-PICO
Parts:
- U2: footprint ESP32-PICO-D4:PQFN50P700X700X104-49N -> Package_DFN_QFN:QFN-48-1EP_7x7mm_P0.5mm_EP5.3x5.3mm
